File: macropad-pcb.kicad_pcb (KiCad board)
At the start: 2 copper layers, 34 parts, among them SW1 SW_Push, U1 ATmega32U4-A, Y1 16MHz

Commit message: Did minor changes on pin assignment on the PCB
Parts:
- turned C3 to -90 degrees
- turned U1 to 90 degrees
Connections:
- U1 pad 10: COL2 -> unconnected-(U1-Pad10)
- U1 pad 19: ROW2 -> unconnected-(U1-Pad19)
- U1 pad 21: ROW1 -> unconnected-(U1-Pad21)
- U1 pad 22: ROW0 -> unconnected-(U1-Pad22)
- U1 pad 28: COL1 -> unconnected-(U1-Pad28)
- U1 pad 30: COL0 -> unconnected-(U1-Pad30)
- U1 pad 36: unconnected-(U1-Pad36) -> COL2
- U1 pad 37: unconnected-(U1-Pad37) -> COL1
- U1 pad 38: unconnected-(U1-Pad38) -> COL0
- U1 pad 39: unconnected-(U1-Pad39) -> ROW2
- U1 pad 40: unconnected-(U1-Pad40) -> ROW1
- U1 pad 41: unconnected-(U1-Pad41) -> ROW0
