File: macropad-pcb.kicad_sch (KiCad schematic)
At the start: 14 parts, among them SW1 SW_Push, U1 ATmega32U4-A, Y1 16MHz

Commit message: Making the PCB
Parts:
- added D1, D2, D3, D4, D5, D6, D7, D8, D9: D_Small, Diode_SMD:D_SOD-123, symbol Device:D_Small
- added F1: 500mA, Fuse:Fuse_1206_3216Metric, symbol Device:Polyfuse_Small
- added MX1, MX2, MX3, MX4, MX5, MX6, MX7, MX8, MX9: MX-NoLED, MX_Alps_Hybrid:MX-1U, symbol MX_Alps_Hybrid:MX-NoLED
- added USB1: Molex-0548190589, random-keyboard-parts:Molex-0548190589, symbol random-keyboard-parts:Molex-0548190589
- C1, C2, C3, C4, C5, C6, C7: footprint (none) -> Capacitor_SMD:C_0805_2012Metric
- R1, R2, R3, R4: footprint (none) -> Resistor_SMD:R_0805_2012Metric
- SW1: footprint (none) -> random-keyboard-parts:SKQG-1155865
- Y1: footprint (none) -> Crystal:Crystal_SMD_3225-4Pin_3.2x2.5mm
Connections:
- net +5V: now also F1.2
- net D+: now also USB1.3 (D+)
- net D-: now also USB1.4 (D-)
- net GND: now also USB1.1 (GND), USB1.6 (SHIELD)
- net COL2: now reaches U1.10 (PB2)
- net COL2: now also MX3.1 (COL), MX6.1 (COL), MX9.1 (COL)
- net ROW2: now reaches U1.19 (PD1)
- net ROW2: now also D7.1 (K), D8.1 (K), D9.1 (K)
- net ROW1: now reaches U1.21 (PD3)
- net ROW1: now also D4.1 (K), D5.1 (K), D6.1 (K)
- net ROW0: now reaches U1.22 (PD5)
- net ROW0: now also D1.1 (K), D2.1 (K), D3.1 (K)
- net COL1: now reaches U1.28 (PB4)
- net COL1: now also MX2.1 (COL), MX5.1 (COL), MX8.1 (COL)
- net COL0: now reaches U1.30 (PB6)
- net COL0: now also MX1.1 (COL), MX4.1 (COL), MX7.1 (COL)
- new net: D7.2 (A), MX7.2 (ROW)
- new net: D2.2 (A), MX2.2 (ROW)
- new net: D9.2 (A), MX9.2 (ROW)
- new net: D5.2 (A), MX5.2 (ROW)
- new net: D1.2 (A), MX1.2 (ROW)
- new net: D4.2 (A), MX4.2 (ROW)
- new net: D8.2 (A), MX8.2 (ROW)
- new net: D6.2 (A), MX6.2 (ROW)
- new net: D3.2 (A), MX3.2 (ROW)
- new net VCC: F1.1, USB1.5 (VBUS)

Commit message: Did minor changes on pin assignment on the PCB
Connections:
- net COL0: now also U1.38 (PF5); no longer U1.30 (PB6)
- net COL1: now also U1.37 (PF6); no longer U1.28 (PB4)
- net COL2: now also U1.36 (PF7); no longer U1.10 (PB2)
- net ROW0: now also U1.41 (PF0); no longer U1.22 (PD5)
- net ROW1: now also U1.40 (PF1); no longer U1.21 (PD3)
- net ROW2: now also U1.39 (PF4); no longer U1.19 (PD1)
Changed lines of the file:
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@@
-    (stroke (width 0) (type default) (color 0 0 0 0))
-  )
-  (wire (pts (xy 102.87 44.45) (xy 111.76 44.45))
     (stroke (width 0) (type default) (color 0 0 0 0))
   )
@@
     (stroke (width 0) (type default) (color 0 0 0 0))
   )
-  (wire (pts (xy 102.87 82.55) (xy 111.76 82.55))
-    (stroke (width 0) (type default) (color 0 0 0 0))
-  )
   (wire (pts (xy 102.87 92.71) (xy 111.76 92.71))
     (stroke (width 0) (type default) (color 0 0 0 0))
@@
     (stroke (width 0) (type default) (color 0 0 0 0))
   )
-  (wire (pts (xy 102.87 72.39) (xy 111.76 72.39))
-    (stroke (width 0) (type default) (color 0 0 0 0))
-  )
   (wire (pts (xy 57.15 59.69) (xy 72.39 59.69))
     (stroke (width 0) (type default) (color 0 0 0 0))
@@
     (stroke (width 0) (type default) (color 0 0 0 0))
   )
+  (wire (pts (xy 102.87 105.41) (xy 110.49 105.41))
+    (stroke (width 0) (type default) (color 0 0 0 0))
+  )
   (wire (pts (xy 34.29 110.49) (xy 39.37 110.49))
     (stroke (width 0) (type default) (color 0 0 0 0))
@@
     (stroke (width 0) (type default) (color 0 0 0 0))
   )
+  (wire (pts (xy 102.87 100.33) (xy 110.49 100.33))
+    (stroke (width 0) (type default) (color 0 0 0 0))
+  )
   (wire (pts (xy 90.17 30.48) (xy 87.63 30.48))
     (stroke (width 0) (type default) (color 0 0 0 0))
@@
     (stroke (width 0) (type default) (color 0 0 0 0))
   )
+  (wire (pts (xy 102.87 102.87) (xy 110.49 102.87))
+    (stroke (width 0) (type default) (color 0 0 0 0))
+  )
   (wire (pts (xy 196.85 53.34) (xy 200.66 53.34))
     (stroke (width 0) (type default) (color 0 0 0 0))
@@
     (stroke (width 0) (type default) (color 0 0 0 0))
   )
-  (wire (pts (xy 102.87 77.47) (xy 111.76 77.47))
-    (stroke (width 0) (type default) (color 0 0 0 0))
-  )
   (wire (pts (xy 181.61 81.28) (xy 181.61 90.17))
     (stroke (width 0) (type default) (color 0 0 0 0))
@@
     (stroke (width 0) (type default) (color 0 0 0 0))
   )
+  (wire (pts (xy 102.87 110.49) (xy 110.49 110.49))
+    (stroke (width 0) (type default) (color 0 0 0 0))
+  )
   (wire (pts (xy 87.63 30.48) (xy 85.09 30.48))
     (stroke (width 0) (type default) (color 0 0 0 0))
@@
     (stroke (width 0) (type default) (color 0 0 0 0))
   )
+  (wire (pts (xy 102.87 113.03) (xy 110.49 113.03))
+    (stroke (width 0) (type default) (color 0 0 0 0))
+  )
   (wire (pts (xy 190.5 100.33) (xy 190.5 104.14))
     (stroke (width 0) (type default) (color 0 0 0 0))
@@
     (stroke (width 0) (type default) (color 0 0 0 0))
   )
+  (wire (pts (xy 102.87 107.95) (xy 110.49 107.95))
+    (stroke (width 0) (type default) (color 0 0 0 0))
+  )
   (wire (pts (xy 190.5 138.43) (xy 194.31 138.43))
     (stroke (width 0) (type default) (color 0 0 0 0))
@@
     (stroke (width 0) (type default) (color 0 0 0 0))
   )
-  (wire (pts (xy 102.87 49.53) (xy 111.76 49.53))
-    (stroke (width 0) (type default) (color 0 0 0 0))
-  )
   (wire (pts (xy 201.93 58.42) (xy 201.93 60.96))
     (stroke (width 0) (type default) (color 0 0 0 0))
@@
   )
   (wire (pts (xy 207.01 95.25) (xy 210.82 95.25))
-    (stroke (width 0) (type default) (color 0 0 0 0))
-  )
-  (wire (pts (xy 102.87 54.61) (xy 111.76 54.61))
     (stroke (width 0) (type default) (color 0 0 0 0))
   )
@@
     )
   )
-  (global_label "COL0" (shape input) (at 111.76 54.61 0) (fields_autoplaced)
-    (effects (font (size 1.27 1.27)) (justify left))
-    (property "Intersheet References" "${INTERSHEET_REFS}" (id 0) (at 119.0112 54.5306 0)
-      (effects (font (size 1.27 1.27)) (justify left) hide)
-    )
-  )
-  (global_label "COL1" (shape input) (at 111.76 49.53 0) (fields_autoplaced)
-    (effects (font (size 1.27 1.27)) (justify left))
-    (property "Intersheet References" "${INTERSHEET_REFS}" (id 0) (at 119.0112 49.4506 0)
+  (global_label "COL0" (shape input) (at 110.49 107.95 0) (fields_autoplaced)
+    (effects (font (size 1.27 1.27)) (justify left))
+    (property "Intersheet References" "${INTERSHEET_REFS}" (id 0) (at 117.7412 107.8706 0)
+      (effects (font (size 1.27 1.27)) (justify left) hide)
+    )
+  )
+  (global_label "COL1" (shape input) (at 110.49 110.49 0) (fields_autoplaced)
+    (effects (font (size 1.27 1.27)) (justify left))
+    (property "Intersheet References" "${INTERSHEET_REFS}" (id 0) (at 117.7412 110.4106 0)
       (effects (font (size 1.27 1.27)) (justify left) hide)
     )
@@
     )
   )
-  (global_label "COL2" (shape input) (at 111.76 44.45 0) (fields_autoplaced)
-    (effects (font (size 1.27 1.27)) (justify left))
-    (property "Intersheet References" "${INTERSHEET_REFS}" (id 0) (at 119.0112 44.3706 0)
+  (global_label "COL2" (shape input) (at 110.49 113.03 0) (fields_autoplaced)
+    (effects (font (size 1.27 1.27)) (justify left))
+    (property "Intersheet References" "${INTERSHEET_REFS}" (id 0) (at 117.7412 112.9506 0)
       (effects (font (size 1.27 1.27)) (justify left) hide)
     )
@@
     )
   )
-  (global_label "ROW1" (shape input) (at 111.76 77.47 0) (fields_autoplaced)
-    (effects (font (size 1.27 1.27)) (justify left))
-    (property "Intersheet References" "${INTERSHEET_REFS}" (id 0) (at 119.4345 77.3906 0)
-      (effects (font (size 1.27 1.27)) (justify left) hide)
-    )
-  )
-  (global_label "ROW0" (shape input) (at 111.76 82.55 0) (fields_autoplaced)
-    (effects (font (size 1.27 1.27)) (justify left))
-    (property "Intersheet References" "${INTERSHEET_REFS}" (id 0) (at 119.4345 82.4706 0)
-      (effects (font (size 1.27 1.27)) (justify left) hide)
-    )
-  )
-  (global_label "ROW2" (shape input) (at 111.76 72.39 0) (fields_autoplaced)
-    (effects (font (size 1.27 1.27)) (justify left))
-    (property "Intersheet References" "${INTERSHEET_REFS}" (id 0) (at 119.4345 72.3106 0)
-      (effects (font (size 1.27 1.27)) (justify left) hide)
-    )
+  (global_label "ROW1" (shape input) (at 110.49 102.87 0) (fields_autoplaced)
+    (effects (font (size 1.27 1.27)) (justify left))
+    (property "Intersheet References" "${INTERSHEET_REFS}" (id 0) (at 118.1645 102.7906 0)
+      (effects (font (size 1.27 1.27)) (justify left) hide)
+    )
+  )
+  (global_label "ROW0" (shape input) (at 110.49 100.33 0) (fields_autoplaced)
+    (effects (font (size 1.27 1.27)) (justify left))
+    (property "Intersheet References" "${INTERSHEET_REFS}" (id 0) (at 118.1645 100.2506 0)
+      (effects (font (size 1.27 1.27)) (justify left) hide)
+    )
+  )
+  (global_label "ROW2" (shape input) (at 110.49 105.41 0) (fields_autoplaced)
+    (effects (font (size 1.27 1.27)) (justify left))
+    (property "Intersheet References" "${INTERSHEET_REFS}" (id 0) (at 118.1645 105.3306 0)
+      (effects (font (size 1.27 1.27)) (justify left) hide)
+    )

Commit message: Add submodules for digikey-kicad-library library
Parts:
- removed F1: 500mA, Fuse:Fuse_1206_3216Metric, symbol Device:Polyfuse_Small
- removed R2, R3: 22, Resistor_SMD:R_0805_2012Metric, symbol Device:R_Small
- removed USB1: Molex-0548190589, random-keyboard-parts:Molex-0548190589, symbol random-keyboard-parts:Molex-0548190589
- added R? (x2): 22, symbol Device:R
- added USB?: HRO-TYPE-C-31-M-12, symbol Type-C:HRO-TYPE-C-31-M-12
Connections:
- net D+: now also U1.4 (D+), R?.2
- net D-: now also U1.3 (D-), R?.2
- new net: R?.1, USB?.6 (DP1), USB?.8 (DP2)
- new net: R?.1, USB?.5 (DN2), USB?.7 (DN1)
